File: Remote PCB V2/Remote PCB V2.kicad_pcb (KiCad board)
At the start: 2 copper layers, 14 parts, among them SW1 SW_Push, SW2 SW_Push, SW3 SW_Push, SW4 SW_Push, SW5 SW_Push

Commit message: V3
Parts:
- moved VBATT1 72.0 mm to (77.9, 65.3), turned to 180 degrees
- moved R2 63.5 mm to (73.8, 65.7), turned to 180 degrees
- moved DWM1 62.6 mm to (95.2, 66.0)
- moved C2 62.2 mm to (105.7, 58.5)
- moved R1 62.2 mm to (105.3, 63.1)
- moved SW2 62.1 mm to (80.2, 3.75)
- moved SW4 62.1 mm to (80.2, 33.8)
- moved SW1 62.1 mm to (68.7, 27.5)
- moved U2 61.7 mm to (62.2, 62.3)
- moved SW3 61.7 mm to (80.2, 18.8)
- moved R4 61.0 mm to (86.1, 65.0), turned to -90 degrees
- moved SW5 58.5 mm to (99.2, 27.5), turned to 90 degrees
- moved R3 50.7 mm to (69.3, 65.7), turned to 180 degrees
- moved GND 42.2 mm to (64.6, 65.3), turned to 180 degrees
- renumbered GND1 to GND
Connections:
- U2 pad 10: DOWN -> RIGHT
- U2 pad 11: STOP -> DOWN
- U2 pad 12: UP -> STOP
- U2 pad 13: LEFT -> UP
- U2 pad 14: unconnected-(U2-12-Pad14) -> LEFT
- U2 pad 3: CS -> VBATT_DIV
- U2 pad 9: VBATT_DIV -> CS
Routing:
- net +3V3: track 0.00 -> 57.8 mm, vias 0 -> 2
- net UP: track 0.00 -> 55.9 mm
- net RIGHT: track 0.00 -> 40.6 mm
- net STOP: track 0.00 -> 40.1 mm
- net LEFT: track 0.00 -> 31.9 mm
- net RST: track 0.00 -> 27.1 mm, vias 0 -> 2
- net VBATT: track 0.00 -> 25.1 mm, vias 0 -> 2
- net DOWN: track 0.00 -> 24.8 mm
- net CLK: track 0.00 -> 19.1 mm, vias 0 -> 2
- net MISO: track 0.00 -> 15.9 mm, vias 0 -> 2
- net MOSI: track 0.00 -> 15.1 mm, vias 0 -> 2
- net GND: track 0.00 -> 10.2 mm, vias 0 -> 3
- net IRQ: track 0.00 -> 9.58 mm
- net CS: track 0.00 -> 7.59 mm
- net VBATT_DIV: track 0.00 -> 7.15 mm
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- added copper zone on B.Cu, net GND
- added copper zone on F.Cu, net GND
Other:
- board outline added: 48 x 67.1 mm
- board text added: "10k"
- board text added: "1k"
- board text added: "1uF"
- board text added: "200k"
- board text added: "600k"
- board text added: "Follow-me Golf Trolley Remote V2.0"
- board text added: "VBATT"
